Commit message: fix: gz 中机械臂倾倒 + mujoco 加载完整场景 + rviz 显示问题
- URDF 加 world dummy link + world_joint(fixed): URDF->SDF 后 base_link 固定
  到 world, 修复 gz 中整机自由浮动倾倒 (与 mujoco MJCF 固定 base 一致)
- demo.launch.py: 加 /clock bridge (gz 内 CM use_sim_time 需要), rviz 延迟
  8s 启动避免 Fixed Frame 竞态; 删兜底 static TF (由 rsp 发布 world->base_link)
- mujoco 默认加载 scene.xml (含地板/灯光完整场景), 可用
  mujoco_model_path:= 覆盖
- SRDF 删 virtual_joint (URDF 根已为 world)
- view.rviz: rviz2 回写的窗口布局

验证: world->base_link 恒 [0,0,0]; none/gz/mujoco 3 控制器 active;
MoveIt PLAN_RESULT error_code=1 points=5

File: src/so101_bringup/urdf/so101.urdf.xacro (robot description, xacro)
@@ -3,5 +3,5 @@
   <!-- sim: none | gazebo | mujoco -->
   <xacro:arg name="sim" default="none"/>
-  <xacro:arg name="mujoco_model_path" default="$(find so101_sim)/mujoco/so101_new_calib.xml"/>
+  <xacro:arg name="mujoco_model_path" default="$(find so101_sim)/mujoco/scene.xml"/>
   <xacro:include filename="$(find so101_description)/urdf/so101.urdf"/>
   <xacro:include filename="$(find so101_sim)/urdf/so101.ros2_control.xacro"/>

File: src/so101_description/urdf/so101.urdf (robot description, URDF)
Before this commit: robot so101, 8 links, 7 joints
Links:
- added link world
Joints:
- added joint world_joint: type fixed, parent world, child base_link, origin xyz=0 0 0 rpy=0 0 0
