Commit message: feat: 力矩控制模型 (xxx_torque) + libs/so101_robotics 学习库 + 对齐验证 --torque
- MJCF/URDF 力矩版: motor actuator ±3.35 Nm, 运动学与位置版 100% 一致
- effort 接口宏 so101_joint_interfaces_effort + controllers_torque.yaml
- libs/so101_robotics: fk/jacobian/ik/dynamics/trajectory/control/constraints/sim
  (pinocchio↔MuJoCo 双引擎交叉验证, hatchling wheel 打包)
- verify_model_alignment.py --torque, 报告全 PASS (FK max 0.0025mm)

File: src/so101_sim/urdf/so101.ros2_control.xacro (robot description, xacro)
@@ -51,3 +51,47 @@
     <xacro:joint_if jname="gripper"/>
   </xacro:macro>
+  <!-- torque 模式: 6 个关节的 effort command + position/velocity state 接口
+       (plan/robotics.md Phase 0, 力矩控制学习版) -->
+  <xacro:macro name="so101_joint_interfaces_effort">
+    <joint name="shoulder_pan">
+      <command_interface name="effort"/>
+      <state_interface name="position"/>
+      <state_interface name="velocity"/>
+    </joint>
+    <joint name="shoulder_lift">
+      <command_interface name="effort"/>
+      <state_interface name="position"/>
+      <state_interface name="velocity"/>
+    </joint>
+    <joint name="elbow_flex">
+      <command_interface name="effort"/>
+      <state_interface name="position"/>
+      <state_interface name="velocity"/>
+    </joint>
+    <joint name="wrist_flex">
+      <command_interface name="effort"/>
+      <state_interface name="position"/>
+      <state_interface name="velocity"/>
+    </joint>
+    <joint name="wrist_roll">
+      <command_interface name="effort"/>
+      <state_interface name="position"/>
+      <state_interface name="velocity"/>
+    </joint>
+    <joint name="gripper">
+      <command_interface name="effort"/>
+      <state_interface name="position"/>
+      <state_interface name="velocity"/>
+    </joint>
+  </xacro:macro>
+  <!-- sim:=mujoco + ctrl_mode:=torque : 加载 scene_torque.xml (motor actuator) -->
+  <xacro:macro name="so101_ros2_control_mujoco_torque" params="name mujoco_model_path">
+    <ros2_control name="${name}" type="system">
+      <hardware>
+        <plugin>mujoco_ros2_control/MujocoSystemInterface</plugin>
+        <param name="mujoco_model">${mujoco_model_path}</param>
+      </hardware>
+      <xacro:so101_joint_interfaces_effort/>
+    </ros2_control>
+  </xacro:macro>
 </robot>
