Commit message: feat: 实机控制模块（so101_hardware 插件 + real:=true 数字孪生 + 命名姿势采集 + 退出归位）
- src/so101_hardware: C++ SystemInterface 实机插件, vendor SCServo SDK;
  标定 YAML 驱动电机 ID/量程, rad↔raw 全行程线性映射, 无零位要求(从当前位置起步);
  激活读不全拒绝激活(防零位冒充); on_deactivate 缓速回启动位姿(parking_ 让路
  + 轮询到位再失能, 回程≤2s); per-motor invert 备用
- launch: real:=true(默认 false), real+mujoco=标准 controller_manager 控实机 +
  mujoco_twin 纯显示; real+gazebo 报错; move_group sim/real/port/calibration 全链透传
- src/so101_sim/mujoco_twin.py: 数字孪生节点(launch_passive + /joint_states 镜像)
- scripts: setup_convert_lerobot_calibration(标定转换+欠扫体检+自动发现全部标定目录)
  / setup_capture_named_pose(力矩失能手摆→命名→SRDF 文本级幂等插入+named_poses.yaml)
- MoveIt 真机调参: allowed_start_tolerance 0.05; SRDF 禁用 lower_arm-shoulder 折叠碰撞
- shoulder_lift 限位手动估计放宽至 ±1.91986(全链 6 处同步+标注, todo/to_real_joint_calibration.md)
- 测试 38 项(契约+xacro 渲染+真实 MJCF/标定集成)

File: models/so101_new_calib.urdf (robot description, URDF)
Before this commit: robot so101_new_calib, 8 links, 7 joints
Joints:
- joint shoulder_lift: limit lower=-1.74533 upper=1.74533 effort=10 velocity=10 -> lower=-1.91986 upper=1.91986 effort=10 velocity=10

File: src/so101_bringup/urdf/so101.urdf.xacro (robot description, xacro)
@@ -1,18 +1,32 @@
 <?xml version="1.0"?>
 <robot xmlns:xacro="http://www.ros.org/wiki/xacro" name="so101">
-  <!-- sim: none | gazebo | mujoco -->
+  <!-- sim: none | gazebo | mujoco; real: true 时 ros2_control 换实机插件 (workflow/plan/setup_hardware.md) -->
   <xacro:arg name="sim" default="none"/>
+  <xacro:arg name="real" default="false"/>
   <xacro:arg name="mujoco_model_path" default="$(find so101_sim)/mujoco/scene.xml"/>
+  <xacro:arg name="port" default="/dev/ttyACM0"/>
+  <xacro:arg name="calibration_file" default="$(find so101_hardware)/config/motor_calibration.yaml"/>
   <xacro:include filename="$(find so101_description)/urdf/so101.urdf"/>
   <xacro:include filename="$(find so101_sim)/urdf/so101.ros2_control.xacro"/>
+  <xacro:include filename="$(find so101_hardware)/urdf/so101.ros2_control_real.xacro"/>
   <xacro:property name="sim" value="$(arg sim)"/>
-  <xacro:if value="${sim == 'none'}">
-    <xacro:so101_ros2_control_mock name="so101"/>
+  <xacro:property name="real" value="$(arg real)"/>
+  <!-- real:=true: 实机插件接管 ros2_control (sim:=mujoco 时 MuJoCo 仅作数字孪生显示)
+       注意: xacro property 求值会把 arg 的 "true"/"false" 自动转成 bool,
+       必须用 ${real} 布尔判断, ${real == 'true'} 字符串比较恒为 False (pitfalls/setup-hardware.md) -->
+  <xacro:if value="${real}">
+    <xacro:so101_ros2_control_real
+        name="so101" port="$(arg port)" calibration_file="$(arg calibration_file)"/>
   </xacro:if>
-  <xacro:if value="${sim == 'gazebo'}">
-    <xacro:so101_ros2_control_gazebo name="so101"/>
-  </xacro:if>
-  <xacro:if value="${sim == 'mujoco'}">
-    <xacro:so101_ros2_control_mujoco name="so101" mujoco_model_path="$(arg mujoco_model_path)"/>
-  </xacro:if>
+  <xacro:unless value="${real}">
+    <xacro:if value="${sim == 'none'}">
+      <xacro:so101_ros2_control_mock name="so101"/>
+    </xacro:if>
+    <xacro:if value="${sim == 'gazebo'}">
+      <xacro:so101_ros2_control_gazebo name="so101"/>
+    </xacro:if>
+    <xacro:if value="${sim == 'mujoco'}">
+      <xacro:so101_ros2_control_mujoco name="so101" mujoco_model_path="$(arg mujoco_model_path)"/>
+    </xacro:if>
+  </xacro:unless>
 </robot>

File: src/so101_description/urdf/so101.urdf (robot description, URDF)
Before this commit: robot so101, 9 links, 8 joints
Joints:
- joint shoulder_lift: limit lower=-1.74533 upper=1.74533 effort=10 velocity=10 -> lower=-1.91986 upper=1.91986 effort=10 velocity=10
